Commit message: Change names

File: urdf/oakd.urdf.xacro (robot description, xacro)
@@ -3,5 +3,5 @@
     <xacro:macro name="oakd" params="name:=oakd parent_link *origin model:=pro">
         <xacro:include
-            filename="$(find gazebo_project)/urdf/common_properties.urdf.xacro" />
+            filename="$(find gazebo_environment)/urdf/common_properties.urdf.xacro" />
         <xacro:property name="mass" value="0.061" />
         <xacro:property name="baseline" value="0.075" />
@@ -24,5 +24,5 @@
                 <geometry>
                     <mesh
-                        filename="package://gazebo_project/meshes/${name}_${model}.dae"
+                        filename="package://gazebo_environment/meshes/${name}_${model}.dae"
                         scale="1 1 1" />
                 </geometry>

File: urdf/robot.urdf (robot description, URDF)
Before this commit: robot robot, 8 links, 7 joints
Links:
- link link_chassis: geometry collision box size=2.4 1.0 1.0; visual mesh filename=package://gazebo_environment/meshes/smart_car.obj scale=0.012 0.012 0.013

File: urdf/tutorial_robot.urdf (robot description, URDF)
Before this commit: robot robot, 8 links, 7 joints
Links:
- link link_chassis: geometry collision box size=2.4 1.0 1.0; visual mesh filename=package://gazebo_environment/meshes/smart_car.obj scale=0.012 0.012 0.013
