Commit message: add: navsat publisher added.

File: urdf/navsat.urdf.xacro (robot description, xacro)
@@ -1,10 +1,10 @@
 <?xml version="1.0"?>
 <robot xmlns:xacro="http://ros.org/wiki/xacro">
-    <xacro:macro name="imu" params="name parent_link *origin namespace update_rate:=30">
+    <xacro:macro name="navsat" params="name parent_link *origin namespace update_rate:=1">
         <xacro:include
             filename="$(find gazebo_environment)/urdf/common_properties.urdf.xacro" />
-        <xacro:property name="base_frame" value="${name}_imu_frame" />
+        <xacro:property name="base_frame" value="${name}_navsat_frame" />
         <!-- Base frame -->
-        <joint name="${name}_imu_joint" type="fixed">
+        <joint name="${name}_navsat_joint" type="fixed">
             <parent link="${parent_link}" />
             <child link="${base_frame}" />
@@ -16,16 +16,15 @@
         <!-- Gazebo links and joints -->
         <gazebo>
-            <plugin filename="ignition-gazebo-imu-system"
-            name="ignition::gazebo::systems::Imu">
+            <plugin
+            filename="ignition-gazebo-navsat-system"
+            name="ignition::gazebo::systems::NavSat">
             </plugin>
         </gazebo>
         <gazebo reference="${base_frame}">
-            <sensor name="imu_sensor" type="imu">
-                <always_on>1</always_on>
-                <update_rate>${update_rate}</update_rate>
-                <visualize>true</visualize>
-                <topic>${namespace}/sensors/${name}/imu</topic>
+            <sensor name="navsat_sensor" type="navsat">
+            <always_on>1</always_on>
+            <update_rate>${update_rate}</update_rate>
+            <topic>${namespace}/sensors/${name}/navsat</topic>
             </sensor>
-            <xacro:material_darkgray />
         </gazebo>
         <gazebo reference="${name}_navsat_joint">

File: urdf/sac.urdf.xacro (robot description, xacro)
@@ -3,4 +3,5 @@
   <xacro:arg name="namespace" default=""/>
   <xacro:include filename="$(find gazebo_environment)/urdf/imu.urdf.xacro" />
+  <xacro:include filename="$(find gazebo_environment)/urdf/navsat.urdf.xacro" />
   <xacro:include filename="$(find gazebo_environment)/urdf/camera.urdf.xacro" />
   <xacro:include filename="$(find gazebo_environment)/urdf/common_properties.urdf.xacro" />
@@ -191,4 +192,21 @@
     <origin xyz="0.0 0.0 0.0" rpy="0.0 0.0 0.0" />
   </xacro:imu>
+<!-- NavSat -->
+  <xacro:navsat name="navsat" parent_link="link_chassis" namespace="$(arg namespace)">
+    <origin xyz="0.0 0.0 0.0" rpy="0.0 0.0 0.0" />
+  </xacro:navsat>
+  <!-- <gazebo>
+    <plugin
+      filename="ignition-gazebo-navsat-system"
+      name="ignition::gazebo::systems::NavSat">
+    </plugin>
+  </gazebo>
+  <gazebo reference="link_chassis">
+    <sensor name="navsat_sensor" type="navsat">
+      <always_on>1</always_on>
+      <update_rate>1</update_rate>
+      <topic>/sensors/navsat</topic>
+    </sensor>
+  </gazebo> -->
   <!-- Ackermann steering plugin -->
   <gazebo>
@@ -218,17 +236,3 @@
       name="ignition::gazebo::systems::JointStatePublisher" />
   </gazebo>
-  <!-- NavSat -->
-  <gazebo>
-    <plugin
-      filename="ignition-gazebo-navsat-system"
-      name="ignition::gazebo::systems::NavSat">
-    </plugin>
-  </gazebo>
-  <gazebo reference="link_chassis">
-    <sensor name="navsat_sensor" type="navsat">
-      <always_on>1</always_on>
-      <update_rate>1</update_rate>
-      <topic>navsat</topic>
-    </sensor>
-  </gazebo>
 </robot>
