Commit message: add: camera imu add. Launch file generilized. Topics are changed.

File: urdf/camera.urdf.xacro (robot description, xacro)
@@ -1,7 +1,7 @@
 <?xml version="1.0"?>
 <robot xmlns:xacro="http://ros.org/wiki/xacro">
-    <xacro:macro name="oakd" params="name:=oakd parent_link *origin model:=pro">
-        <xacro:include
-            filename="$(find gazebo_environment)/urdf/common_properties.urdf.xacro" />
+    <xacro:macro name="camera" params="name parent_link *origin namespace">
+        <xacro:include filename="$(find gazebo_environment)/urdf/common_properties.urdf.xacro" />
+        <xacro:include filename="$(find gazebo_environment)/urdf/imu.urdf.xacro" />
         <xacro:property name="mass" value="0.061" />
         <xacro:property name="baseline" value="0.075" />
@@ -13,5 +13,5 @@
         <xacro:property name="collision_offset_y" value="${0*cm2m}" />
         <xacro:property name="collision_offset_z" value="${-0.5*cm2m}" />
-        <xacro:property name="base_frame" value="oakd_link" />
+        <xacro:property name="base_frame" value="${name}_camera_link" />
         <!-- Base frame -->
         <joint name="${name}_joint" type="fixed">
@@ -24,5 +24,5 @@
                 <geometry>
                     <mesh
-                        filename="package://gazebo_environment/meshes/${name}_${model}.dae"
+                        filename="package://gazebo_environment/meshes/oakd_pro.dae"
                         scale="1 1 1" />
                 </geometry>
@@ -92,13 +92,15 @@
         </joint>
         <!-- IMU -->
-        <link name="${name}_imu_frame">
-            <xacro:inertial_dummy />
-        </link>
-        <joint name="${name}_imu_joint" type="fixed">
-            <parent link="${base_frame}" />
-            <child link="${name}_imu_frame" />
-            <origin xyz="0 0 0" rpy="-${M_PI/2} 0 -${M_PI/2}" />
-        </joint>
+        <xacro:imu name="${name}" parent_link="${base_frame}" namespace="${namespace}">
+            <origin xyz="0.0 0.0 0.0" rpy="-${M_PI/2} 0 -${M_PI/2}" />
+        </xacro:imu>
         <!-- Gazebo links and joints -->
+        <gazebo>
+            <plugin
+                filename="gz-sim-sensors-system"
+                name="gz::sim::systems::Sensors">
+                <render_engine>ogre2</render_engine>
+            </plugin>
+        </gazebo>
         <gazebo reference="${name}_rgb_camera_frame">
             <sensor name="rgbd_camera" type="rgbd_camera">
@@ -118,4 +120,5 @@
                 <update_rate>30</update_rate>
                 <visualize>true</visualize>
+                <topic>${namespace}/sensors/${name}</topic>
             </sensor>
             <xacro:material_darkgray />

File: urdf/sac.urdf.xacro (robot description, xacro)
@@ -1,9 +1,11 @@
 <?xml version="1.0"?>
-<robot name="robot" xmlns:xacro="http://ros.org/wiki/xacro">
-  <xacro:include filename="$(find gazebo_environment)/urdf/oakd.urdf.xacro" />
+<robot name="sac" xmlns:xacro="http://ros.org/wiki/xacro">
+  <xacro:arg name="namespace" default=""/>
+  <xacro:include filename="$(find gazebo_environment)/urdf/imu.urdf.xacro" />
+  <xacro:include filename="$(find gazebo_environment)/urdf/camera.urdf.xacro" />
   <xacro:include filename="$(find gazebo_environment)/urdf/common_properties.urdf.xacro" />
-  <xacro:property name="oakd_pro_x_offset" value="2.0" />
-  <xacro:property name="oakd_pro_y_offset" value="0.0" />
-  <xacro:property name="oakd_pro_z_offset" value="3.0" />
+  <xacro:property name="camera_x_offset" value="2.0" />
+  <xacro:property name="camera_y_offset" value="0.0" />
+  <xacro:property name="camera_z_offset" value="3.0" />
   <link name="base_link">
     <xacro:cuboid_inertia mass="1.0" x="0.1" y="0.1" z="0.1" />
@@ -71,8 +73,4 @@
   <!-- Rear Right Wheel -->
   <link name="rear_right_wheel">
-    <!-- <inertial>
-      <mass value="11.0" />
-      <inertia ixx="0.58" ixy="0.0" iyy="0.33" ixz="0.0" iyz="0.0" izz="0.33" />
-    </inertial> -->
     <xacro:inertial_cylinder mass="11.0" radius="0.25" length="0.15" />
     <visual name="rear_right_wheel_visual">
@@ -106,8 +104,4 @@
   <!-- Front Left Wheel -->
   <link name="front_left_wheel">
-    <!-- <inertial>
-      <mass value="11.0" />
-      <inertia ixx="0.58" ixy="0.0" iyy="0.33" ixz="0.0" iyz="0.0" izz="0.33" />
-    </inertial> -->
     <xacro:inertial_cylinder mass="11.0" radius="0.25" length="0.15" />
     <visual name="front_left_wheel_visual">
@@ -150,8 +144,4 @@
   <!-- Front Right Wheel -->
   <link name="front_right_wheel">
-    <!-- <inertial>
-      <mass value="11.0" />
-      <inertia ixx="0.58" ixy="0.0" iyy="0.33" ixz="0.0" iyz="0.0" izz="0.33" />
-    </inertial> -->
     <xacro:inertial_cylinder mass="11.0" radius="0.25" length="0.15" />
     <visual name="front_right_wheel_visual">
@@ -176,8 +166,4 @@
   </link>
   <link name="front_right_wheel_steering_link">
-    <!-- <inertial>
-      <mass value="1.0" />
-      <inertia ixx="0.58" ixy="0.0" iyy="0.33" ixz="0.0" iyz="0.0" izz="0.33" />
-    </inertial> -->
     <xacro:cuboid_inertia mass="1.0" x="0.1" y="0.1" z="0.1" />
   </link>
@@ -197,7 +183,12 @@
     <joint_properties damping="1.0" friction="1.0" />
   </joint>
-  <xacro:oakd model="pro" parent_link="link_chassis">
-    <origin xyz="${oakd_pro_x_offset} ${oakd_pro_y_offset} ${oakd_pro_z_offset}" rpy="0.0 0.9 0.0" />
-  </xacro:oakd>
+<!-- Camera Plugin -->
+  <xacro:camera name="front_camera" parent_link="link_chassis" namespace="$(arg namespace)">
+    <origin xyz="${camera_x_offset} ${camera_y_offset} ${camera_z_offset}" rpy="0.0 0.9 0.0" />
+  </xacro:camera>
+<!-- IMU Plugin -->
+<xacro:imu name="middle_imu" parent_link="link_chassis" namespace="$(arg namespace)">
+    <origin xyz="0.0 0.0 0.0" rpy="0.0 0.0 0.0" />
+  </xacro:imu>
   <!-- Ackermann steering plugin -->
   <gazebo>
@@ -227,25 +218,4 @@
       name="ignition::gazebo::systems::JointStatePublisher" />
   </gazebo>
-  <!-- IMU Plugin -->
-  <gazebo>
-    <plugin filename="ignition-gazebo-imu-system"
-      name="ignition::gazebo::systems::Imu">
-    </plugin>
-  </gazebo>
-  <gazebo reference="link_chassis">
-    <sensor name="imu_sensor" type="imu">
-      <always_on>1</always_on>
-      <update_rate>20</update_rate>
-      <visualize>true</visualize>
-      <topic>imu</topic>
-    </sensor>
-  </gazebo>
-  <gazebo>
-    <plugin
-      filename="gz-sim-sensors-system"
-      name="gz::sim::systems::Sensors">
-      <render_engine>ogre2</render_engine>
-    </plugin>
-  </gazebo>
   <!-- NavSat -->
   <gazebo>

Commit message: add: Launch problems are solved. but multi spawn problem did not solved. Also depth camera did not work well.

File: urdf/camera.urdf.xacro (robot description, xacro)
@@ -24,5 +24,5 @@
                 <geometry>
                     <mesh
-                        filename="package://gazebo_environment/meshes/oakd_pro.dae"
+                        filename="$(find gazebo_environment)/meshes/oakd_pro.dae"
                         scale="1 1 1" />
                 </geometry>

File: urdf/sac.urdf.xacro (robot description, xacro)
@@ -1,4 +1,4 @@
 <?xml version="1.0"?>
-<robot name="sac" xmlns:xacro="http://ros.org/wiki/xacro">
+<robot name="$(arg namespace)" xmlns:xacro="http://ros.org/wiki/xacro">
   <xacro:arg name="namespace" default=""/>
   <xacro:include filename="$(find gazebo_environment)/urdf/imu.urdf.xacro" />
@@ -9,4 +9,11 @@
   <xacro:property name="camera_y_offset" value="0.0" />
   <xacro:property name="camera_z_offset" value="3.0" />
+  <link name="base_footprint">
+  </link>
+  <joint name="joint_base_footprint_base_link" type="fixed">
+    <origin rpy="0 0 0" xyz="0 0 0" />
+    <child link="base_link" />
+    <parent link="base_footprint" />
+  </joint>
   <link name="base_link">
     <xacro:cuboid_inertia mass="1.0" x="0.1" y="0.1" z="0.1" />
@@ -21,5 +28,5 @@
       <origin rpy="1.57 0 1.57" xyz="0 0 0" />
       <geometry>
-        <mesh filename="package://gazebo_environment/meshes/smart_car.obj"
+        <mesh filename="$(find gazebo_environment)/meshes/smart_car.obj"
           scale="0.012 0.012
         0.013" />
@@ -189,5 +196,5 @@
   </xacro:camera>
 <!-- IMU Plugin -->
-<xacro:imu name="middle_imu" parent_link="link_chassis" namespace="$(arg namespace)">
+  <xacro:imu name="middle_imu" parent_link="link_chassis" namespace="$(arg namespace)">
     <origin xyz="0.0 0.0 0.0" rpy="0.0 0.0 0.0" />
   </xacro:imu>
@@ -196,24 +203,11 @@
     <origin xyz="0.0 0.0 0.0" rpy="0.0 0.0 0.0" />
   </xacro:navsat>
-  <!-- <gazebo>
-    <plugin
-      filename="ignition-gazebo-navsat-system"
-      name="ignition::gazebo::systems::NavSat">
-    </plugin>
-  </gazebo>
-  <gazebo reference="link_chassis">
-    <sensor name="navsat_sensor" type="navsat">
-      <always_on>1</always_on>
-      <update_rate>1</update_rate>
-      <topic>/sensors/navsat</topic>
-    </sensor>
-  </gazebo> -->
   <!-- Ackermann steering plugin -->
   <gazebo>
     <plugin filename="ignition-gazebo-ackermann-steering-system"
       name="ignition::gazebo::systems::AckermannSteering">
-      <topic>/cmd_vel</topic>
+      <topic>$(arg namespace)/actuators/cmd_vel</topic>
       <odom_publish_frequency>10</odom_publish_frequency>
-      <odom_topic>odom</odom_topic>
+      <odom_topic>$(arg namespace)/calculations/steering_odom</odom_topic>
       <left_joint>front_left_wheel_rotating_joint</left_joint>
       <right_joint>front_right_wheel_rotating_joint</right_joint>

Commit message: add:  lidar3d added to xacro and bridge is added to launch file. fix: Camera pointcloud axis error fixed.

File: urdf/camera.urdf.xacro (robot description, xacro)
@@ -53,5 +53,5 @@
         </link>
         <joint name="${name}_rgb_camera_optical_joint" type="fixed">
-            <origin xyz="0 0 0" rpy="-${M_PI/2} 0.0 -${M_PI/2}" />
+            <origin xyz="0 0 0" rpy="0.0 0.0 0.0" />
             <parent link="${name}_rgb_camera_frame" />
             <child link="${name}_rgb_camera_optical_frame" />

File: urdf/sac.urdf.xacro (robot description, xacro)
@@ -5,8 +5,6 @@
   <xacro:include filename="$(find gazebo_environment)/urdf/navsat.urdf.xacro" />
   <xacro:include filename="$(find gazebo_environment)/urdf/camera.urdf.xacro" />
+  <xacro:include filename="$(find gazebo_environment)/urdf/lidar3d.urdf.xacro" />
   <xacro:include filename="$(find gazebo_environment)/urdf/common_properties.urdf.xacro" />
-  <xacro:property name="camera_x_offset" value="2.0" />
-  <xacro:property name="camera_y_offset" value="0.0" />
-  <xacro:property name="camera_z_offset" value="3.0" />
   <link name="base_footprint">
   </link>
@@ -193,5 +191,5 @@
 <!-- Camera Plugin -->
   <xacro:camera name="front_camera" parent_link="link_chassis" namespace="$(arg namespace)">
-    <origin xyz="${camera_x_offset} ${camera_y_offset} ${camera_z_offset}" rpy="0.0 0.9 0.0" />
+    <origin xyz="2 0 3" rpy="0.0 0.9 0.0" />
   </xacro:camera>
 <!-- IMU Plugin -->
@@ -199,8 +197,12 @@
     <origin xyz="0.0 0.0 0.0" rpy="0.0 0.0 0.0" />
   </xacro:imu>
-<!-- NavSat -->
+<!-- NavSat Plugin -->
   <xacro:navsat name="navsat" parent_link="link_chassis" namespace="$(arg namespace)">
     <origin xyz="0.0 0.0 0.0" rpy="0.0 0.0 0.0" />
   </xacro:navsat>
+<!-- 3D Lidar Plugin -->
+  <xacro:lidar3d name="front_3d_lidar" parent_link="link_chassis" namespace="$(arg namespace)">
+    <origin xyz="-0.3 0.0 1.6" rpy="0 0 0" />
+  </xacro:lidar3d>
   <!-- Joint states plugin -->
   <gazebo>
