Commit message: feat: headless mode, real Sonoma GPS location, meshes via package://
- sonoma.launch.py: gui:=false runs only the Gazebo server with
  --headless-rendering (no window or display needed, sensors still
  render). Default stays gui:=true.
- Set GZ_SIM_RESOURCE_PATH as well: Gazebo Harmonic no longer reads
  IGN_GAZEBO_RESOURCE_PATH.
- sonoma.sdf: spherical_coordinates at the real Sonoma Raceway (was an
  Istanbul placeholder). Origin and heading (0.83 deg) come from fitting
  the model's track surface to the OpenStreetMap raceway ways; median
  error ~5 m, about half the track width. GPS now lines up with maps.
- navsat at 10 Hz instead of 1 Hz.
- Car mesh as package://gazebo_environment/..., so Foxglove/Lichtblick
  can load it through foxglove_bridge; Gazebo resolves it through the
  resource path.

Co-Authored-By: Claude Opus 5.5 <noreply@anthropic.com>

File: urdf/sac.urdf.xacro (robot description, xacro)
@@ -26,5 +26,5 @@
       <origin rpy="1.57 0 1.57" xyz="0 0 0" />
       <geometry>
-        <mesh filename="$(find gazebo_environment)/meshes/smart_car.obj"
+        <mesh filename="package://gazebo_environment/meshes/smart_car.obj"
           scale="0.012 0.012
         0.013" />
@@ -173,5 +173,6 @@
   </xacro:imu>
 <!-- NavSat Plugin -->
-  <xacro:navsat name="navsat" parent_link="link_chassis" namespace="$(arg namespace)">
+  <!-- 10 Hz like a typical GNSS receiver; at 1 Hz a map view barely moves -->
+  <xacro:navsat name="navsat" parent_link="link_chassis" namespace="$(arg namespace)" update_rate="10">
     <origin xyz="0.0 0.0 0.0" rpy="0.0 0.0 0.0" />
   </xacro:navsat>

Commit message: feat: roof rack with the sensors, as on the real car
From photos and measurements of the real car:
- Aluminium-profile roof rack (1.2 x 1.1 m, 40 mm profiles on 5 cm feet,
  cross bar through the middle; sizes estimated from photos), visual only.
- VLP-16 on a post on the cross bar, in the middle of the rack, its base
  20 cm above the roof (measured): lidar frame at z 1.793 m.
- ZED 2 level on a 10 cm ball head in the middle of the front bar (was
  behind the windshield).
- GNSS antenna pucks at both ends of the front bar; the simulated receiver
  uses the left one.
The lowest lidar beams (-15..-3 deg) hit the rack, camera and antennas
0.5-0.8 m away, as they would on the real car.

Co-Authored-By: Claude Opus 5.5 <noreply@anthropic.com>

File: urdf/sac.urdf.xacro (robot description, xacro)
@@ -18,4 +18,5 @@
   <xacro:include filename="$(find gazebo_environment)/urdf/zed2.urdf.xacro" />
   <xacro:include filename="$(find gazebo_environment)/urdf/lidar3d.urdf.xacro" />
+  <xacro:include filename="$(find gazebo_environment)/urdf/roof_rack.urdf.xacro" />
   <!-- ============ Vehicle parameters (smart fortwo W453; not measured) ============ -->
   <xacro:property name="wheel_base" value="1.873" />      <!-- front axle to rear axle [m] -->
@@ -40,12 +41,25 @@
   <xacro:property name="max_acceleration" value="3.0" />  <!-- [m/s^2] -->
   <xacro:property name="max_deceleration" value="7.0" />  <!-- braking [m/s^2] -->
-  <!-- Sensor mounts, relative to base_footprint / link_chassis (same origin; not measured) -->
-  <!-- ZED 2 behind the top of the windshield, tilted down to see the road -->
-  <xacro:property name="camera_xyz" value="0.45 0 1.40" />
-  <xacro:property name="camera_pitch" value="0.15" />     <!-- [rad], positive tilts down -->
-  <!-- VLP-16 on the roof; the lidar frame is its optical centre, 37.7 mm above the roof -->
-  <xacro:property name="lidar_xyz" value="-0.2 0 ${1.555 + 0.0377}" />
-  <xacro:property name="imu_xyz" value="0 0 0.5" />       <!-- about the centre of mass -->
-  <xacro:property name="gnss_xyz" value="-0.5 0 1.555" /> <!-- antenna on the roof -->
+  <!-- Roof rack (aluminium profiles, estimated from photos of the real car) -->
+  <xacro:property name="roof_z" value="${body_top}" />
+  <xacro:property name="rack_front_x" value="0.50" />       <!-- front bar, at the top of the windshield -->
+  <xacro:property name="rack_rear_x" value="-0.70" />
+  <xacro:property name="rack_half_width" value="0.55" />
+  <xacro:property name="rack_clearance" value="0.05" />     <!-- feet: roof to the bottom of the profiles -->
+  <xacro:property name="rack_profile" value="0.04" />       <!-- 40 x 40 mm profile -->
+  <xacro:property name="rack_top_z" value="${roof_z + rack_clearance + rack_profile}" />
+  <xacro:property name="rack_mid_x" value="${(rack_front_x + rack_rear_x) / 2}" />
+  <!-- Sensor mounts, relative to base_footprint / link_chassis (same origin) -->
+  <!-- ZED 2 on a 10 cm ball head in the middle of the front bar, level -->
+  <xacro:property name="camera_xyz" value="${rack_front_x} 0 ${rack_top_z + 0.10}" />
+  <xacro:property name="camera_pitch" value="0.0" />      <!-- [rad], positive tilts down -->
+  <!-- VLP-16 on a post on the cross bar, in the middle of the rack, its base 20 cm above
+       the roof (measured); the lidar frame is its optical centre, 37.7 mm above the base -->
+  <xacro:property name="lidar_base_above_roof" value="0.20" />
+  <xacro:property name="lidar_xyz" value="${rack_mid_x} 0 ${roof_z + lidar_base_above_roof + 0.0377}" />
+  <!-- GNSS antennas at both ends of the front bar; the simulated receiver uses the left one -->
+  <xacro:property name="gnss_antenna_y" value="${rack_half_width - 0.05}" />
+  <xacro:property name="gnss_xyz" value="${rack_front_x} ${gnss_antenna_y} ${rack_top_z + 0.07}" />
+  <xacro:property name="imu_xyz" value="0 0 0.5" />       <!-- about the centre of mass (not measured) -->
   <!-- ============================== Body ============================== -->
   <link name="base_footprint" />
@@ -151,4 +165,8 @@
   <xacro:front_wheel side="right" y="${-front_track / 2}" />
   <!-- ============================== Sensors ============================== -->
+  <xacro:roof_rack parent_link="link_chassis" roof_z="${roof_z}" front_x="${rack_front_x}"
+    rear_x="${rack_rear_x}" half_width="${rack_half_width}" clearance="${rack_clearance}"
+    profile="${rack_profile}" post_height="${lidar_base_above_roof - rack_clearance - rack_profile}"
+    antenna_y="${gnss_antenna_y}" />
   <xacro:zed2 name="front_camera" parent_link="link_chassis" namespace="$(arg namespace)">
     <origin xyz="${camera_xyz}" rpy="0 ${camera_pitch} 0" />

Commit message: fix: fit the roof rack to the roof and to the real rack's width
The rack was 1.1 m wide and reached from the windshield to behind the
roof, so it hung in the air over the curved edges. The roof of the body
mesh is flat only from x 0 to -0.9 m and y +-0.45 m. The real rack is
about 0.75 m wide: in the front photo its front bar is 4.3 times the
ZED 2's 175 mm.
Now: 0.9 x 0.75 m, front bar at the top of the windshield, feet on the
roof. The lidar (middle of the rack, base 20 cm above the roof) sees the
car in 1.5% of its points instead of 18%.

Co-Authored-By: Claude Opus 5.5 <noreply@anthropic.com>

File: urdf/sac.urdf.xacro (robot description, xacro)
@@ -41,12 +41,14 @@
   <xacro:property name="max_acceleration" value="3.0" />  <!-- [m/s^2] -->
   <xacro:property name="max_deceleration" value="7.0" />  <!-- braking [m/s^2] -->
-  <!-- Roof rack (aluminium profiles, estimated from photos of the real car) -->
-  <xacro:property name="roof_z" value="${body_top}" />
-  <xacro:property name="rack_front_x" value="0.50" />       <!-- front bar, at the top of the windshield -->
-  <xacro:property name="rack_rear_x" value="-0.70" />
-  <xacro:property name="rack_half_width" value="0.55" />
+  <!-- Roof rack (aluminium profiles). Width from photos of the real car, scaled by the ZED 2's
+       known 175 mm width; length fits the flat part of the roof (x 0 to -0.9, y +-0.45). -->
+  <xacro:property name="roof_z" value="${body_top}" />      <!-- highest point of the roof -->
+  <xacro:property name="rack_base_z" value="1.53" />       <!-- roof height under the rack's feet -->
+  <xacro:property name="rack_front_x" value="0.0" />        <!-- front bar, at the top of the windshield -->
+  <xacro:property name="rack_rear_x" value="-0.9" />
+  <xacro:property name="rack_half_width" value="0.375" />
   <xacro:property name="rack_clearance" value="0.05" />     <!-- feet: roof to the bottom of the profiles -->
   <xacro:property name="rack_profile" value="0.04" />       <!-- 40 x 40 mm profile -->
-  <xacro:property name="rack_top_z" value="${roof_z + rack_clearance + rack_profile}" />
+  <xacro:property name="rack_top_z" value="${rack_base_z + rack_clearance + rack_profile}" />
   <xacro:property name="rack_mid_x" value="${(rack_front_x + rack_rear_x) / 2}" />
   <!-- Sensor mounts, relative to base_footprint / link_chassis (same origin) -->
@@ -59,5 +61,5 @@
   <xacro:property name="lidar_xyz" value="${rack_mid_x} 0 ${roof_z + lidar_base_above_roof + 0.0377}" />
   <!-- GNSS antennas at both ends of the front bar; the simulated receiver uses the left one -->
-  <xacro:property name="gnss_antenna_y" value="${rack_half_width - 0.05}" />
+  <xacro:property name="gnss_antenna_y" value="${rack_half_width - 0.03}" />
   <xacro:property name="gnss_xyz" value="${rack_front_x} ${gnss_antenna_y} ${rack_top_z + 0.07}" />
   <xacro:property name="imu_xyz" value="0 0 0.5" />       <!-- about the centre of mass (not measured) -->
@@ -165,7 +167,7 @@
   <xacro:front_wheel side="right" y="${-front_track / 2}" />
   <!-- ============================== Sensors ============================== -->
-  <xacro:roof_rack parent_link="link_chassis" roof_z="${roof_z}" front_x="${rack_front_x}"
+  <xacro:roof_rack parent_link="link_chassis" roof_z="${rack_base_z}" front_x="${rack_front_x}"
     rear_x="${rack_rear_x}" half_width="${rack_half_width}" clearance="${rack_clearance}"
-    profile="${rack_profile}" post_height="${lidar_base_above_roof - rack_clearance - rack_profile}"
+    profile="${rack_profile}" post_height="${roof_z + lidar_base_above_roof - rack_top_z}"
     antenna_y="${gnss_antenna_y}" />
   <xacro:zed2 name="front_camera" parent_link="link_chassis" namespace="$(arg namespace)">

Commit message: feat: second IMU at the front; middle_imu back in the middle
- middle_imu in the middle of the car again (0, 0, 0.5).
- front_imu over the front axle (0.936, 0, 0.5), on the chassis, same
  BMI085-like noise, bridged lazily on /sac/sensors/front_imu/imu.

Co-Authored-By: Claude Opus 5.5 <noreply@anthropic.com>

File: urdf/sac.urdf.xacro (robot description, xacro)
@@ -66,6 +66,8 @@
   <xacro:property name="gnss_antenna_y" value="${rack_half_width - 0.03}" />
   <xacro:property name="gnss_xyz" value="${rack_front} ${gnss_antenna_y} 0.07" />
-  <!-- IMU at the front of the car, on the centre line over the front axle (not measured) -->
-  <xacro:property name="imu_xyz" value="${wheel_base / 2} 0 0.5" />
+  <!-- Two IMUs on the chassis, on the centre line (not measured): one in the middle of the
+       car, one over the front axle -->
+  <xacro:property name="middle_imu_xyz" value="0 0 0.5" />
+  <xacro:property name="front_imu_xyz" value="${wheel_base / 2} 0 0.5" />
   <!-- ============================== Body ============================== -->
   <link name="base_footprint" />
@@ -178,7 +180,9 @@
     <origin xyz="${camera_xyz}" rpy="0 ${camera_pitch} 0" />
   </xacro:zed2>
-  <!-- Named middle_imu for its topic, /sac/sensors/middle_imu/imu -->
   <xacro:imu name="middle_imu" parent_link="link_chassis" namespace="$(arg namespace)">
-    <origin xyz="${imu_xyz}" rpy="0 0 0" />
+    <origin xyz="${middle_imu_xyz}" rpy="0 0 0" />
+  </xacro:imu>
+  <xacro:imu name="front_imu" parent_link="link_chassis" namespace="$(arg namespace)">
+    <origin xyz="${front_imu_xyz}" rpy="0 0 0" />
   </xacro:imu>
   <!-- 10 Hz like a typical GNSS receiver -->

Commit message: feat: third IMU over the rear axle
back_imu at (-0.936, 0, 0.5) on the chassis, same noise as the others,
bridged lazily on /sac/sensors/back_imu/imu.

Co-Authored-By: Claude Opus 5.5 <noreply@anthropic.com>

File: urdf/sac.urdf.xacro (robot description, xacro)
@@ -66,8 +66,9 @@
   <xacro:property name="gnss_antenna_y" value="${rack_half_width - 0.03}" />
   <xacro:property name="gnss_xyz" value="${rack_front} ${gnss_antenna_y} 0.07" />
-  <!-- Two IMUs on the chassis, on the centre line (not measured): one in the middle of the
-       car, one over the front axle -->
+  <!-- Three IMUs on the chassis, on the centre line (not measured): in the middle of the
+       car, over the front axle and over the rear axle -->
   <xacro:property name="middle_imu_xyz" value="0 0 0.5" />
   <xacro:property name="front_imu_xyz" value="${wheel_base / 2} 0 0.5" />
+  <xacro:property name="back_imu_xyz" value="${-wheel_base / 2} 0 0.5" />
   <!-- ============================== Body ============================== -->
   <link name="base_footprint" />
@@ -186,4 +187,7 @@
     <origin xyz="${front_imu_xyz}" rpy="0 0 0" />
   </xacro:imu>
+  <xacro:imu name="back_imu" parent_link="link_chassis" namespace="$(arg namespace)">
+    <origin xyz="${back_imu_xyz}" rpy="0 0 0" />
+  </xacro:imu>
   <!-- 10 Hz like a typical GNSS receiver -->
   <xacro:navsat name="navsat" parent_link="roof_rack" namespace="$(arg namespace)" update_rate="10">
