Commit message: feat: REP 105 TF (map -> odom -> base_footprint), optional; roof_lidar
- odometry_tf publishes map -> odom (identity) and odom -> base_footprint
  from Gazebo's exact pose, instead of world -> base_footprint. The launch
  argument ground_truth_tf:=false leaves both to a localization such as
  robot_localization's EKF, which would otherwise give base_footprint two
  parents. The track marker is in map.
- The steering plugin's wheel odometry is in odom (was steering_odom), so
  an EKF can take it as it is.
- The lidar is on the middle of the roof rack, not at the front: renamed
  front_3d_lidar -> roof_lidar, topic /sac/sensors/roof_lidar/points and
  frame roof_lidar_frame (the macro no longer doubles "lidar" in names).
- readme: TF section.

Checked: default chain map <- odom <- base_footprint <- ... <- roof_lidar_frame;
with ground_truth_tf:=false no map/odom is published.

Co-Authored-By: Claude Opus 5.5 <noreply@anthropic.com>

File: urdf/lidar3d.urdf.xacro (robot description, xacro)
@@ -14,6 +14,6 @@
     <xacro:property name="lidar_noise" value="0.015" />
     <xacro:macro name="lidar3d" params="name parent_link *origin namespace update_rate:=10">
-        <xacro:property name="base_frame" value="${name}_lidar_frame" />
-        <joint name="${name}_lidar_joint" type="fixed">
+        <xacro:property name="base_frame" value="${name}_frame" />
+        <joint name="${name}_joint" type="fixed">
             <parent link="${parent_link}" />
             <child link="${base_frame}" />
@@ -31,5 +31,5 @@
         </link>
         <gazebo reference="${base_frame}">
-            <sensor name="${name}_lidar_sensor" type="gpu_lidar">
+            <sensor name="${name}_sensor" type="gpu_lidar">
                 <always_on>true</always_on>
                 <update_rate>${update_rate}</update_rate>
@@ -62,5 +62,5 @@
             </sensor>
         </gazebo>
-        <gazebo reference="${name}_lidar_joint">
+        <gazebo reference="${name}_joint">
             <preserveFixedJoint>true</preserveFixedJoint>
         </gazebo>

File: urdf/sac.urdf.xacro (robot description, xacro)
@@ -194,5 +194,5 @@
     <origin xyz="${gnss_xyz}" rpy="0 0 0" />
   </xacro:navsat>
-  <xacro:lidar3d name="front_3d_lidar" parent_link="roof_rack" namespace="$(arg namespace)">
+  <xacro:lidar3d name="roof_lidar" parent_link="roof_rack" namespace="$(arg namespace)">
     <origin xyz="${lidar_xyz}" rpy="0 0 0" />
   </xacro:lidar3d>
@@ -233,5 +233,6 @@
       <odom_topic>$(arg namespace)/calculations/steering_odom</odom_topic>
       <tf_topic>$(arg namespace)/tf/steering_odom</tf_topic>
-      <frame_id>steering_odom</frame_id>
+      <!-- Wheel odometry in the odom frame (REP 105), ready for an EKF -->
+      <frame_id>odom</frame_id>
       <child_frame_id>base_footprint</child_frame_id>
     </plugin>
