Commit message: feat: smart fortwo body, ZED 2 camera, VLP-16 lidar; MIT license
Match the model to the real car's hardware:
- Vehicle: Mercedes smart fortwo (W453) datasheet values: 1.873 m
  wheelbase, 1.469/1.430 m track, 0.30 m wheels, ~880 kg, 0.6 rad
  steering (6.95 m turning circle), rear-wheel drive like the smart,
  20 m/s top speed, 3 m/s^2 acceleration. The body mesh (already a smart)
  is scaled to 2.695 x 1.663 x 1.555 m. Measured: 25 m/s commanded ->
  accelerates at 3 m/s^2 and holds 20.00 m/s; 0.1 rad/s -> 0.106 rad/s.
- Camera: Stereolabs ZED 2 (120 mm baseline, 110 deg HFOV, 0.3-20 m
  depth, IMU) replaces the OAK-D Pro. Frame names follow the ZED ROS 2
  wrapper (front_camera_left_camera_optical_frame, _imu_link, ...); the
  colour image is clipped at 500 m, depth at 20 m. Simulated at 1280x720,
  30 Hz. The 12 MB OAK-D mesh is removed.
- Lidar: VLP-16 beam pattern (16 channels over +-15 deg, 1800 samples at
  10 Hz, 1.5 cm noise). The mesh was drawn at twice its size (scale 0.002
  for a mesh in mm); the link origin is now the optical centre.
- imu macro takes an optional frame name.
- LICENSE (MIT), package.xml and setup.py license.

Co-Authored-By: Claude Opus 5.5 <noreply@anthropic.com>

File: urdf/imu.urdf.xacro (robot description, xacro)
@@ -2,6 +2,7 @@
 <!-- IMU on a fixed link. Needs the Imu system in the world. -->
 <robot xmlns:xacro="http://ros.org/wiki/xacro">
-    <xacro:macro name="imu" params="name parent_link *origin namespace update_rate:=100">
-        <xacro:property name="base_frame" value="${name}_imu_frame" />
+    <xacro:macro name="imu" params="name parent_link *origin namespace update_rate:=100 frame:=''">
+        <!-- Frame name: <name>_imu_frame unless given -->
+        <xacro:property name="base_frame" value="${frame if frame else name + '_imu_frame'}" />
         <joint name="${name}_imu_joint" type="fixed">
             <parent link="${parent_link}" />

File: urdf/lidar3d.urdf.xacro (robot description, xacro)
@@ -1,15 +1,16 @@
 <?xml version="1.0"?>
 <!--
-  3D lidar (GPU ray casting) on a fixed link, publishing a point cloud.
+  Velodyne VLP-16 (GPU ray casting) on a fixed link, publishing a point cloud.
+  The link origin is the sensor's optical centre, 37.7 mm above its base.
   Needs the Sensors system in the world.
-  The visual is a Velodyne VLP-16, but the beam pattern below is not a VLP-16 (that has
-  16 channels over +-15 deg). Set it to the real lidar's values.
 -->
 <robot xmlns:xacro="http://ros.org/wiki/xacro">
-    <xacro:property name="lidar_horizontal_samples" value="360" />
-    <xacro:property name="lidar_vertical_samples" value="40" />
-    <xacro:property name="lidar_vertical_half_angle" value="0.186" />  <!-- [rad] -->
+    <!-- VLP-16 datasheet: 16 channels over +-15 deg, 0.2 deg steps at 10 Hz, 100 m, +-3 cm -->
+    <xacro:property name="lidar_horizontal_samples" value="1800" />
+    <xacro:property name="lidar_vertical_samples" value="16" />
+    <xacro:property name="lidar_vertical_half_angle" value="${15 * pi / 180}" />
     <xacro:property name="lidar_min_range" value="0.5" />
     <xacro:property name="lidar_max_range" value="100.0" />
+    <xacro:property name="lidar_noise" value="0.015" />
     <xacro:macro name="lidar3d" params="name parent_link *origin namespace update_rate:=10">
         <xacro:property name="base_frame" value="${name}_lidar_frame" />
@@ -22,8 +23,8 @@
             <xacro:inertial_dummy />
             <visual>
-                <!-- The mesh is Y-up and in millimetres -->
-                <origin xyz="0 0 0" rpy="${pi/2} 0 ${pi}" />
+                <!-- The mesh is Y-up, in millimetres, with its origin at the base -->
+                <origin xyz="0 0 -0.0377" rpy="${pi/2} 0 ${pi}" />
                 <geometry>
-                    <mesh filename="package://gazebo_environment/meshes/velodyne-vlp16.stl" scale="0.002 0.002 0.002" />
+                    <mesh filename="package://gazebo_environment/meshes/velodyne-vlp16.stl" scale="0.001 0.001 0.001" />
                 </geometry>
             </visual>
@@ -56,5 +57,5 @@
                         <type>gaussian</type>
                         <mean>0.0</mean>
-                        <stddev>0.01</stddev>
+                        <stddev>${lidar_noise}</stddev>
                     </noise>
                 </lidar>

File: urdf/sac.urdf.xacro (robot description, xacro)
@@ -1,8 +1,10 @@
 <?xml version="1.0"?>
 <!--
-  SAC: Ackermann-steered car with a front RGB-D camera, a 3D lidar, an IMU and a GNSS
-  receiver, for Gazebo Harmonic.
+  SAC: a Mercedes smart fortwo sized car (rear-wheel drive, Ackermann steering) with a
+  ZED 2 stereo camera, a Velodyne VLP-16 lidar, an IMU and a GNSS receiver, for Gazebo
+  Harmonic.
   All dimensions and limits are properties below, so the model can be matched to the real
-  car in one place. Values marked "not measured" are placeholders.
+  car in one place. Values marked "not measured" come from the smart fortwo (W453)
+  datasheet or are estimates, not from the real car.
   Frames (REP 103/105): x forward, y left, z up. base_footprint lies on the ground under
   the middle of the car; wheels turn in the positive direction when the car drives forward.
@@ -14,29 +16,32 @@
   <xacro:include filename="$(find gazebo_environment)/urdf/imu.urdf.xacro" />
   <xacro:include filename="$(find gazebo_environment)/urdf/navsat.urdf.xacro" />
-  <xacro:include filename="$(find gazebo_environment)/urdf/camera.urdf.xacro" />
+  <xacro:include filename="$(find gazebo_environment)/urdf/zed2.urdf.xacro" />
   <xacro:include filename="$(find gazebo_environment)/urdf/lidar3d.urdf.xacro" />
-  <!-- ===================== Vehicle parameters (not measured) ===================== -->
-  <xacro:property name="wheel_base" value="1.8" />        <!-- front axle to rear axle [m] -->
-  <xacro:property name="track_width" value="1.28" />      <!-- left to right wheel centre [m] -->
-  <xacro:property name="wheel_radius" value="0.25" />
-  <xacro:property name="wheel_width" value="0.15" />
-  <xacro:property name="wheel_mass" value="11.0" />
-  <xacro:property name="steering_limit" value="0.8" />    <!-- [rad] -->
-  <!-- Body, used for collisions and inertia; matches the size of the visual mesh -->
-  <xacro:property name="body_length" value="2.6" />
-  <xacro:property name="body_width" value="1.5" />
-  <xacro:property name="body_bottom" value="0.125" />     <!-- ground clearance [m] -->
-  <xacro:property name="body_top" value="1.44" />
-  <xacro:property name="body_mass" value="500.0" />
+  <!-- ============ Vehicle parameters (smart fortwo W453; not measured) ============ -->
+  <xacro:property name="wheel_base" value="1.873" />      <!-- front axle to rear axle [m] -->
+  <xacro:property name="front_track" value="1.469" />     <!-- left to right wheel centre [m] -->
+  <xacro:property name="rear_track" value="1.430" />
+  <xacro:property name="wheel_radius" value="0.30" />     <!-- 165/65 R15 front, 185/60 R15 rear -->
+  <xacro:property name="wheel_width" value="0.175" />
+  <xacro:property name="wheel_mass" value="15.0" />
+  <!-- 6.95 m turning circle -->
+  <xacro:property name="steering_limit" value="0.6" />    <!-- [rad] -->
+  <!-- Body, used for collisions and inertia -->
+  <xacro:property name="body_length" value="2.695" />
+  <xacro:property name="body_width" value="1.663" />
+  <xacro:property name="body_bottom" value="0.15" />      <!-- ground clearance [m] -->
+  <xacro:property name="body_top" value="1.555" />
+  <xacro:property name="body_mass" value="820.0" />       <!-- ~880 kg kerb weight without wheels -->
   <xacro:property name="max_speed" value="20.0" />        <!-- [m/s] forward -->
-  <xacro:property name="max_reverse_speed" value="10.0" />
-  <xacro:property name="max_acceleration" value="5.0" />  <!-- [m/s^2] -->
+  <xacro:property name="max_reverse_speed" value="5.0" />
+  <xacro:property name="max_acceleration" value="3.0" />  <!-- [m/s^2] -->
   <!-- Sensor mounts, relative to base_footprint / link_chassis (same origin; not measured) -->
-  <!-- Front camera at the top of the windshield, tilted down to see the road -->
-  <xacro:property name="camera_xyz" value="0.5 0 1.35" />
-  <xacro:property name="camera_pitch" value="0.2" />      <!-- [rad], positive tilts down -->
-  <xacro:property name="lidar_xyz" value="-0.3 0 1.6" />
-  <xacro:property name="imu_xyz" value="0 0 0.6" />       <!-- about the centre of mass -->
-  <xacro:property name="gnss_xyz" value="0 0 1.44" />     <!-- antenna on the roof -->
+  <!-- ZED 2 behind the top of the windshield, tilted down to see the road -->
+  <xacro:property name="camera_xyz" value="0.45 0 1.40" />
+  <xacro:property name="camera_pitch" value="0.15" />     <!-- [rad], positive tilts down -->
+  <!-- VLP-16 on the roof; the lidar frame is its optical centre, 37.7 mm above the roof -->
+  <xacro:property name="lidar_xyz" value="-0.2 0 ${1.555 + 0.0377}" />
+  <xacro:property name="imu_xyz" value="0 0 0.5" />       <!-- about the centre of mass -->
+  <xacro:property name="gnss_xyz" value="-0.5 0 1.555" /> <!-- antenna on the roof -->
   <!-- ============================== Body ============================== -->
   <link name="base_footprint" />
@@ -58,8 +63,8 @@
   <link name="link_chassis">
     <visual name="chassis_visual">
-      <!-- The mesh is Y-up and in centimetres -->
+      <!-- A smart fortwo, Y-up; the scale makes it 2.695 x 1.663 x 1.555 m -->
       <origin xyz="0 0 0" rpy="${pi/2} 0 ${pi/2}" />
       <geometry>
-        <mesh filename="package://gazebo_environment/meshes/smart_car.obj" scale="0.012 0.012 0.013" />
+        <mesh filename="package://gazebo_environment/meshes/smart_car.obj" scale="0.0125 0.0129 0.0135" />
       </geometry>
       <material name="white">
@@ -137,12 +142,12 @@
     </joint>
   </xacro:macro>
-  <xacro:rear_wheel side="left" y="${track_width / 2}" />
-  <xacro:rear_wheel side="right" y="${-track_width / 2}" />
-  <xacro:front_wheel side="left" y="${track_width / 2}" />
-  <xacro:front_wheel side="right" y="${-track_width / 2}" />
+  <xacro:rear_wheel side="left" y="${rear_track / 2}" />
+  <xacro:rear_wheel side="right" y="${-rear_track / 2}" />
+  <xacro:front_wheel side="left" y="${front_track / 2}" />
+  <xacro:front_wheel side="right" y="${-front_track / 2}" />
   <!-- ============================== Sensors ============================== -->
-  <xacro:camera name="front_camera" parent_link="link_chassis" namespace="$(arg namespace)">
+  <xacro:zed2 name="front_camera" parent_link="link_chassis" namespace="$(arg namespace)">
     <origin xyz="${camera_xyz}" rpy="0 ${camera_pitch} 0" />
-  </xacro:camera>
+  </xacro:zed2>
   <xacro:imu name="middle_imu" parent_link="link_chassis" namespace="$(arg namespace)">
     <origin xyz="${imu_xyz}" rpy="0 0 0" />
@@ -171,16 +176,16 @@
     </plugin>
   </gazebo>
-  <!-- Front-wheel drive and steering from /<namespace>/actuators/cmd_vel -->
+  <!-- Rear-wheel drive (like the smart) and front steering from /<namespace>/actuators/cmd_vel -->
   <gazebo>
     <plugin filename="gz-sim-ackermann-steering-system" name="gz::sim::systems::AckermannSteering">
       <topic>$(arg namespace)/actuators/cmd_vel</topic>
-      <left_joint>front_left_wheel_rotating_joint</left_joint>
-      <right_joint>front_right_wheel_rotating_joint</right_joint>
+      <left_joint>rear_left_wheel_joint</left_joint>
+      <right_joint>rear_right_wheel_joint</right_joint>
       <left_steering_joint>front_left_wheel_steering_joint</left_steering_joint>
       <right_steering_joint>front_right_wheel_steering_joint</right_steering_joint>
-      <kingpin_width>${track_width}</kingpin_width>
+      <kingpin_width>${front_track}</kingpin_width>
       <steering_limit>${steering_limit}</steering_limit>
       <wheel_base>${wheel_base}</wheel_base>
-      <wheel_separation>${track_width}</wheel_separation>
+      <wheel_separation>${rear_track}</wheel_separation>
       <wheel_radius>${wheel_radius}</wheel_radius>
       <min_velocity>${-max_reverse_speed}</min_velocity>

Commit message: feat: realistic sensor noise, centre of mass, camera rate and braking
- ZED 2 at 15 Hz, one of its modes (was 30): real-time factor with the
  viewer open 0.72 -> 0.95. Gaussian image noise.
- IMU noise and per-run bias from the BMI085 datasheet (ZED 2's IMU),
  measured: gyro 0.0017 rad/s, accel 0.012 m/s^2.
- GNSS noise of a standalone receiver, 1 m horizontal / 1.5 m vertical.
  Gazebo adds horizontal noise in degrees, so it is converted from metres
  (measured 0.94 m north, 0.81 m east, 1.36 m altitude).
- Centre of mass of a rear-engined smart: 40/60 axle load, 0.55 m high.
  Stable: 0.02 rad pitch under braking, 0.02 rad roll in a 17 m turn.
- Braking limit 7 m/s^2, separate from the 3 m/s^2 acceleration.
- VLP-16 stays at its factory mode (1800 samples at 10 Hz); 900 samples
  only exist at 20 Hz, which casts as many rays.
- readme: what is and is not like the real car.

Co-Authored-By: Claude Opus 5.5 <noreply@anthropic.com>

File: urdf/imu.urdf.xacro (robot description, xacro)
@@ -2,4 +2,21 @@
 <!-- IMU on a fixed link. Needs the Imu system in the world. -->
 <robot xmlns:xacro="http://ros.org/wiki/xacro">
+    <!-- Noise of a MEMS IMU like the ZED 2's (Bosch BMI085) at 100 Hz: white noise from the
+         noise densities (0.014 deg/s/sqrt(Hz), 175 ug/sqrt(Hz)) over a 50 Hz bandwidth, and a
+         constant bias drawn once per run -->
+    <xacro:property name="imu_gyro_noise" value="0.0017" />         <!-- [rad/s] -->
+    <xacro:property name="imu_gyro_bias" value="0.0005" />          <!-- [rad/s] -->
+    <xacro:property name="imu_accel_noise" value="0.012" />         <!-- [m/s^2] -->
+    <xacro:property name="imu_accel_bias" value="0.02" />           <!-- [m/s^2] -->
+    <xacro:macro name="imu_axis_noise" params="axis stddev bias">
+        <xacro:element xacro:name="${axis}">
+            <noise type="gaussian">
+                <mean>0.0</mean>
+                <stddev>${stddev}</stddev>
+                <bias_mean>0.0</bias_mean>
+                <bias_stddev>${bias}</bias_stddev>
+            </noise>
+        </xacro:element>
+    </xacro:macro>
     <xacro:macro name="imu" params="name parent_link *origin namespace update_rate:=100 frame:=''">
         <!-- Frame name: <name>_imu_frame unless given -->
@@ -19,4 +36,16 @@
                 <topic>${namespace}/sensors/${name}/imu</topic>
                 <gz_frame_id>${base_frame}</gz_frame_id>
+                <imu>
+                    <angular_velocity>
+                        <xacro:imu_axis_noise axis="x" stddev="${imu_gyro_noise}" bias="${imu_gyro_bias}" />
+                        <xacro:imu_axis_noise axis="y" stddev="${imu_gyro_noise}" bias="${imu_gyro_bias}" />
+                        <xacro:imu_axis_noise axis="z" stddev="${imu_gyro_noise}" bias="${imu_gyro_bias}" />
+                    </angular_velocity>
+                    <linear_acceleration>
+                        <xacro:imu_axis_noise axis="x" stddev="${imu_accel_noise}" bias="${imu_accel_bias}" />
+                        <xacro:imu_axis_noise axis="y" stddev="${imu_accel_noise}" bias="${imu_accel_bias}" />
+                        <xacro:imu_axis_noise axis="z" stddev="${imu_accel_noise}" bias="${imu_accel_bias}" />
+                    </linear_acceleration>
+                </imu>
             </sensor>
         </gazebo>

File: urdf/navsat.urdf.xacro (robot description, xacro)
@@ -3,4 +3,16 @@
      <spherical_coordinates> in the world for real latitude/longitude. -->
 <robot xmlns:xacro="http://ros.org/wiki/xacro">
+    <!-- Error of a standalone (non-RTK) GNSS receiver. Gazebo adds the horizontal noise to
+         latitude and longitude in degrees, so it is converted from metres here. -->
+    <xacro:property name="gnss_horizontal_noise" value="1.0" />   <!-- [m] -->
+    <xacro:property name="gnss_vertical_noise" value="1.5" />     <!-- [m] -->
+    <xacro:property name="gnss_velocity_noise" value="0.05" />    <!-- [m/s] -->
+    <xacro:property name="metres_per_degree" value="111320.0" />
+    <xacro:macro name="gnss_noise" params="stddev">
+        <noise type="gaussian">
+            <mean>0.0</mean>
+            <stddev>${stddev}</stddev>
+        </noise>
+    </xacro:macro>
     <xacro:macro name="navsat" params="name parent_link *origin namespace update_rate:=10">
         <xacro:property name="base_frame" value="${name}_navsat_frame" />
@@ -19,4 +31,22 @@
                 <topic>${namespace}/sensors/${name}/navsat</topic>
                 <gz_frame_id>${base_frame}</gz_frame_id>
+                <navsat>
+                    <position_sensing>
+                        <horizontal>
+                            <xacro:gnss_noise stddev="${gnss_horizontal_noise / metres_per_degree}" />
+                        </horizontal>
+                        <vertical>
+                            <xacro:gnss_noise stddev="${gnss_vertical_noise}" />
+                        </vertical>
+                    </position_sensing>
+                    <velocity_sensing>
+                        <horizontal>
+                            <xacro:gnss_noise stddev="${gnss_velocity_noise}" />
+                        </horizontal>
+                        <vertical>
+                            <xacro:gnss_noise stddev="${gnss_velocity_noise}" />
+                        </vertical>
+                    </velocity_sensing>
+                </navsat>
             </sensor>
         </gazebo>

File: urdf/sac.urdf.xacro (robot description, xacro)
@@ -33,7 +33,11 @@
   <xacro:property name="body_top" value="1.555" />
   <xacro:property name="body_mass" value="820.0" />       <!-- ~880 kg kerb weight without wheels -->
+  <!-- Centre of mass: rear engine, ~40/60 front/rear axle load, low in the car -->
+  <xacro:property name="com_x" value="${-wheel_base / 2 + 0.4 * wheel_base}" />
+  <xacro:property name="com_z" value="0.55" />
   <xacro:property name="max_speed" value="20.0" />        <!-- [m/s] forward -->
   <xacro:property name="max_reverse_speed" value="5.0" />
   <xacro:property name="max_acceleration" value="3.0" />  <!-- [m/s^2] -->
+  <xacro:property name="max_deceleration" value="7.0" />  <!-- braking [m/s^2] -->
   <!-- Sensor mounts, relative to base_footprint / link_chassis (same origin; not measured) -->
   <!-- ZED 2 behind the top of the windshield, tilted down to see the road -->
@@ -79,5 +83,5 @@
     </collision>
     <xacro:inertial_cuboid_with_pose mass="${body_mass}" x="${body_length}" y="${body_width}" z="${body_height}">
-      <origin xyz="0 0 ${body_center_z}" rpy="0 0 0" />
+      <origin xyz="${com_x} 0 ${com_z}" rpy="0 0 0" />
     </xacro:inertial_cuboid_with_pose>
   </link>
@@ -191,5 +195,5 @@
       <min_velocity>${-max_reverse_speed}</min_velocity>
       <max_velocity>${max_speed}</max_velocity>
-      <min_acceleration>${-max_acceleration}</min_acceleration>
+      <min_acceleration>${-max_deceleration}</min_acceleration>
       <max_acceleration>${max_acceleration}</max_acceleration>
       <odom_publish_frequency>10</odom_publish_frequency>

File: urdf/zed2.urdf.xacro (robot description, xacro)
@@ -17,8 +17,11 @@
     <xacro:property name="zed2_min_depth" value="0.3" />
     <xacro:property name="zed2_max_depth" value="20.0" />
-    <!-- Simulated stream: HD720 at 30 Hz (the camera also does 1080p/2K) -->
+    <!-- Simulated stream: HD720 at 15 Hz, one of the camera's modes (it also does 30/60 Hz,
+         1080p and 2K) -->
     <xacro:property name="zed2_width" value="1280" />
     <xacro:property name="zed2_height_px" value="720" />
-    <xacro:property name="zed2_rate" value="30" />
+    <xacro:property name="zed2_rate" value="15" />
+    <!-- Sensor noise of the colour image, as a fraction of the pixel range -->
+    <xacro:property name="zed2_image_noise" value="0.007" />
     <xacro:macro name="zed2" params="name parent_link *origin namespace">
         <!-- Rotation from a body frame (x forward) to an optical frame (z forward) -->
@@ -97,4 +100,9 @@
                         </clip>
                     </depth_camera>
+                    <noise>
+                        <type>gaussian</type>
+                        <mean>0.0</mean>
+                        <stddev>${zed2_image_noise}</stddev>
+                    </noise>
                     <optical_frame_id>${name}_left_camera_optical_frame</optical_frame_id>
                 </camera>

Commit message: refactor: simpler IMU and GNSS frame names
The macros doubled the sensor type in the names. Before the real drivers
are set up to match:
  middle_imu_imu_frame -> middle_imu_frame (front_imu, back_imu too)
  navsat_navsat_frame  -> navsat_frame
Topics are unchanged; the ZED IMU keeps the wrapper's front_camera_imu_link.

Co-Authored-By: Claude Opus 5.5 <noreply@anthropic.com>

File: urdf/imu.urdf.xacro (robot description, xacro)
@@ -20,7 +20,7 @@
     </xacro:macro>
     <xacro:macro name="imu" params="name parent_link *origin namespace update_rate:=100 frame:=''">
-        <!-- Frame name: <name>_imu_frame unless given -->
-        <xacro:property name="base_frame" value="${frame if frame else name + '_imu_frame'}" />
-        <joint name="${name}_imu_joint" type="fixed">
+        <!-- Frame name: <name>_frame unless given -->
+        <xacro:property name="base_frame" value="${frame if frame else name + '_frame'}" />
+        <joint name="${base_frame}_joint" type="fixed">
             <parent link="${parent_link}" />
             <child link="${base_frame}" />
@@ -51,5 +51,5 @@
         </gazebo>
         <!-- Keep the frame as its own link in Gazebo so the sensor reports in it -->
-        <gazebo reference="${name}_imu_joint">
+        <gazebo reference="${base_frame}_joint">
             <preserveFixedJoint>true</preserveFixedJoint>
         </gazebo>

File: urdf/navsat.urdf.xacro (robot description, xacro)
@@ -16,6 +16,6 @@
     </xacro:macro>
     <xacro:macro name="navsat" params="name parent_link *origin namespace update_rate:=10">
-        <xacro:property name="base_frame" value="${name}_navsat_frame" />
-        <joint name="${name}_navsat_joint" type="fixed">
+        <xacro:property name="base_frame" value="${name}_frame" />
+        <joint name="${name}_joint" type="fixed">
             <parent link="${parent_link}" />
             <child link="${base_frame}" />
@@ -51,5 +51,5 @@
             </sensor>
         </gazebo>
-        <gazebo reference="${name}_navsat_joint">
+        <gazebo reference="${name}_joint">
             <preserveFixedJoint>true</preserveFixedJoint>
         </gazebo>
