Commit message: refactor: hang the roof sensors off the rack, IMU at the front
- The camera, lidar and GNSS antenna are children of roof_rack instead of
  link_chassis, like on the real car. The rack frame now sits in the middle
  of the rack on top of the profiles, so their mounts are given (and can
  be measured) relative to the rack; their positions on the car are
  unchanged (camera 0/0/1.72, lidar -0.45/0/1.793, GNSS 0/0.345/1.69).
- IMU on the chassis at the front, on the centre line over the front
  axle (0.936, 0, 0.5). Its name stays middle_imu to keep its topic.

Co-Authored-By: Claude Opus 5.5 <noreply@anthropic.com>

File: urdf/roof_rack.urdf.xacro (robot description, xacro)
@@ -2,19 +2,26 @@
 <!--
   Aluminium-profile roof rack that carries the sensors: a rectangular frame on feet with a
-  cross bar through the middle, a post on the cross bar for the lidar, and two GNSS
-  antenna pucks at the ends of the front bar. Visual only (no collisions), with a small mass.
-  The sizes are estimated from photos of the real car; the sensor mounts in sac.urdf.xacro
-  are computed from them.
+  cross bar through the middle, a post on the cross bar for the lidar, a ball head for the
+  camera and two GNSS antenna pucks at the ends of the front bar. Visual only (no
+  collisions), with a small mass.
+  The rack frame "roof_rack" sits in the middle of the rack, on the top of the profiles
+  (x forward, z up), so sensor mounts can be given, and measured on the real car, relative
+  to the rack. Arguments are in the parent's frame.
 -->
 <robot xmlns:xacro="http://ros.org/wiki/xacro">
     <xacro:macro name="roof_rack" params="parent_link roof_z front_x rear_x half_width clearance profile post_height antenna_y">
         <xacro:property name="length" value="${front_x - rear_x}" />
-        <xacro:property name="mid_x" value="${(front_x + rear_x) / 2}" />
-        <!-- Centre height of the profiles -->
-        <xacro:property name="bar_z" value="${roof_z + clearance + profile / 2}" />
+        <!-- Rack frame in the parent's coordinates -->
+        <xacro:property name="ox" value="${(front_x + rear_x) / 2}" />
+        <xacro:property name="oz" value="${roof_z + clearance + profile}" />
+        <!-- In the rack frame -->
+        <xacro:property name="front" value="${front_x - ox}" />
+        <xacro:property name="rear" value="${rear_x - ox}" />
+        <xacro:property name="bar_z" value="${-profile / 2}" />
+        <xacro:property name="foot_z" value="${-profile - clearance / 2}" />
         <joint name="roof_rack_joint" type="fixed">
             <parent link="${parent_link}" />
             <child link="roof_rack" />
-            <origin xyz="0 0 0" rpy="0 0 0" />
+            <origin xyz="${ox} 0 ${oz}" rpy="0 0 0" />
         </joint>
         <xacro:macro name="rack_box" params="xyz size material:=rack_aluminium">
@@ -29,19 +36,19 @@
         <link name="roof_rack">
             <!-- Frame: front, rear, left, right bars and the cross bar through the middle -->
-            <xacro:rack_box xyz="${front_x} 0 ${bar_z}" size="${profile} ${2 * half_width} ${profile}" />
-            <xacro:rack_box xyz="${rear_x} 0 ${bar_z}" size="${profile} ${2 * half_width} ${profile}" />
-            <xacro:rack_box xyz="${mid_x} ${half_width} ${bar_z}" size="${length} ${profile} ${profile}" />
-            <xacro:rack_box xyz="${mid_x} ${-half_width} ${bar_z}" size="${length} ${profile} ${profile}" />
-            <xacro:rack_box xyz="${mid_x} 0 ${bar_z}" size="${profile} ${2 * half_width} ${profile}" />
+            <xacro:rack_box xyz="${front} 0 ${bar_z}" size="${profile} ${2 * half_width} ${profile}" />
+            <xacro:rack_box xyz="${rear} 0 ${bar_z}" size="${profile} ${2 * half_width} ${profile}" />
+            <xacro:rack_box xyz="0 ${half_width} ${bar_z}" size="${length} ${profile} ${profile}" />
+            <xacro:rack_box xyz="0 ${-half_width} ${bar_z}" size="${length} ${profile} ${profile}" />
+            <xacro:rack_box xyz="0 0 ${bar_z}" size="${profile} ${2 * half_width} ${profile}" />
             <!-- Feet on the roof at the four corners -->
-            <xacro:rack_box xyz="${front_x} ${half_width} ${roof_z + clearance / 2}" size="0.06 0.06 ${clearance}" material="rack_plastic" />
-            <xacro:rack_box xyz="${front_x} ${-half_width} ${roof_z + clearance / 2}" size="0.06 0.06 ${clearance}" material="rack_plastic" />
-            <xacro:rack_box xyz="${rear_x} ${half_width} ${roof_z + clearance / 2}" size="0.06 0.06 ${clearance}" material="rack_plastic" />
-            <xacro:rack_box xyz="${rear_x} ${-half_width} ${roof_z + clearance / 2}" size="0.06 0.06 ${clearance}" material="rack_plastic" />
+            <xacro:rack_box xyz="${front} ${half_width} ${foot_z}" size="0.06 0.06 ${clearance}" material="rack_plastic" />
+            <xacro:rack_box xyz="${front} ${-half_width} ${foot_z}" size="0.06 0.06 ${clearance}" material="rack_plastic" />
+            <xacro:rack_box xyz="${rear} ${half_width} ${foot_z}" size="0.06 0.06 ${clearance}" material="rack_plastic" />
+            <xacro:rack_box xyz="${rear} ${-half_width} ${foot_z}" size="0.06 0.06 ${clearance}" material="rack_plastic" />
             <!-- Lidar post on the cross bar -->
-            <xacro:rack_box xyz="${mid_x} 0 ${bar_z + profile / 2 + post_height / 2}" size="0.03 0.03 ${post_height}" />
+            <xacro:rack_box xyz="0 0 ${post_height / 2}" size="0.03 0.03 ${post_height}" />
             <!-- Ball head under the camera, in the middle of the front bar -->
             <visual>
-                <origin xyz="${front_x} 0 ${bar_z + profile / 2 + 0.05}" rpy="0 0 0" />
+                <origin xyz="${front} 0 0.05" rpy="0 0 0" />
                 <geometry>
                     <cylinder radius="0.02" length="0.10" />
@@ -50,8 +57,8 @@
             </visual>
             <!-- GNSS antenna pucks on blocks at both ends of the front bar -->
-            <xacro:rack_box xyz="${front_x} ${antenna_y} ${bar_z + profile / 2 + 0.02}" size="0.06 0.06 0.04" material="rack_plastic" />
-            <xacro:rack_box xyz="${front_x} ${-antenna_y} ${bar_z + profile / 2 + 0.02}" size="0.06 0.06 0.04" material="rack_plastic" />
+            <xacro:rack_box xyz="${front} ${antenna_y} 0.02" size="0.06 0.06 0.04" material="rack_plastic" />
+            <xacro:rack_box xyz="${front} ${-antenna_y} 0.02" size="0.06 0.06 0.04" material="rack_plastic" />
             <visual>
-                <origin xyz="${front_x} ${antenna_y} ${bar_z + profile / 2 + 0.055}" rpy="0 0 0" />
+                <origin xyz="${front} ${antenna_y} 0.055" rpy="0 0 0" />
                 <geometry>
                     <cylinder radius="0.04" length="0.03" />
@@ -60,5 +67,5 @@
             </visual>
             <visual>
-                <origin xyz="${front_x} ${-antenna_y} ${bar_z + profile / 2 + 0.055}" rpy="0 0 0" />
+                <origin xyz="${front} ${-antenna_y} 0.055" rpy="0 0 0" />
                 <geometry>
                     <cylinder radius="0.04" length="0.03" />
@@ -67,7 +74,11 @@
             </visual>
             <xacro:inertial_cuboid_with_pose mass="8.0" x="${length}" y="${2 * half_width}" z="${profile}">
-                <origin xyz="${mid_x} 0 ${bar_z}" rpy="0 0 0" />
+                <origin xyz="0 0 ${bar_z}" rpy="0 0 0" />
             </xacro:inertial_cuboid_with_pose>
         </link>
+        <!-- Keep the rack as its own link in Gazebo, so the sensors hang off it -->
+        <gazebo reference="roof_rack_joint">
+            <preserveFixedJoint>true</preserveFixedJoint>
+        </gazebo>
     </xacro:macro>
     <material name="rack_aluminium">

File: urdf/sac.urdf.xacro (robot description, xacro)
@@ -52,16 +52,20 @@
   <xacro:property name="rack_top_z" value="${rack_base_z + rack_clearance + rack_profile}" />
   <xacro:property name="rack_mid_x" value="${(rack_front_x + rack_rear_x) / 2}" />
-  <!-- Sensor mounts, relative to base_footprint / link_chassis (same origin) -->
+  <!-- Sensor mounts. The camera, lidar and GNSS antennas are on the roof rack and given
+       relative to its frame (middle of the rack, top of the profiles); the IMU is on the
+       chassis, relative to base_footprint. -->
+  <xacro:property name="rack_front" value="${rack_front_x - rack_mid_x}" />  <!-- front bar, in the rack frame -->
   <!-- ZED 2 on a 10 cm ball head in the middle of the front bar, level -->
-  <xacro:property name="camera_xyz" value="${rack_front_x} 0 ${rack_top_z + 0.10}" />
+  <xacro:property name="camera_xyz" value="${rack_front} 0 0.10" />
   <xacro:property name="camera_pitch" value="0.0" />      <!-- [rad], positive tilts down -->
   <!-- VLP-16 on a post on the cross bar, in the middle of the rack, its base 20 cm above
        the roof (measured); the lidar frame is its optical centre, 37.7 mm above the base -->
   <xacro:property name="lidar_base_above_roof" value="0.20" />
-  <xacro:property name="lidar_xyz" value="${rack_mid_x} 0 ${roof_z + lidar_base_above_roof + 0.0377}" />
+  <xacro:property name="lidar_xyz" value="0 0 ${roof_z + lidar_base_above_roof - rack_top_z + 0.0377}" />
   <!-- GNSS antennas at both ends of the front bar; the simulated receiver uses the left one -->
   <xacro:property name="gnss_antenna_y" value="${rack_half_width - 0.03}" />
-  <xacro:property name="gnss_xyz" value="${rack_front_x} ${gnss_antenna_y} ${rack_top_z + 0.07}" />
-  <xacro:property name="imu_xyz" value="0 0 0.5" />       <!-- about the centre of mass (not measured) -->
+  <xacro:property name="gnss_xyz" value="${rack_front} ${gnss_antenna_y} 0.07" />
+  <!-- IMU at the front of the car, on the centre line over the front axle (not measured) -->
+  <xacro:property name="imu_xyz" value="${wheel_base / 2} 0 0.5" />
   <!-- ============================== Body ============================== -->
   <link name="base_footprint" />
@@ -171,15 +175,16 @@
     profile="${rack_profile}" post_height="${roof_z + lidar_base_above_roof - rack_top_z}"
     antenna_y="${gnss_antenna_y}" />
-  <xacro:zed2 name="front_camera" parent_link="link_chassis" namespace="$(arg namespace)">
+  <xacro:zed2 name="front_camera" parent_link="roof_rack" namespace="$(arg namespace)">
     <origin xyz="${camera_xyz}" rpy="0 ${camera_pitch} 0" />
   </xacro:zed2>
+  <!-- Named middle_imu for its topic, /sac/sensors/middle_imu/imu -->
   <xacro:imu name="middle_imu" parent_link="link_chassis" namespace="$(arg namespace)">
     <origin xyz="${imu_xyz}" rpy="0 0 0" />
   </xacro:imu>
   <!-- 10 Hz like a typical GNSS receiver -->
-  <xacro:navsat name="navsat" parent_link="link_chassis" namespace="$(arg namespace)" update_rate="10">
+  <xacro:navsat name="navsat" parent_link="roof_rack" namespace="$(arg namespace)" update_rate="10">
     <origin xyz="${gnss_xyz}" rpy="0 0 0" />
   </xacro:navsat>
-  <xacro:lidar3d name="front_3d_lidar" parent_link="link_chassis" namespace="$(arg namespace)">
+  <xacro:lidar3d name="front_3d_lidar" parent_link="roof_rack" namespace="$(arg namespace)">
     <origin xyz="${lidar_xyz}" rpy="0 0 0" />
   </xacro:lidar3d>

Commit message: feat: two GNSS antennas; drive from the viewer's Teleop panel
- GNSS: two antennas at opposite rack corners, front right and rear left,
  like the real car: /sac/sensors/navsat_front_right/navsat and
  /sac/sensors/navsat_rear_left/navsat (frames navsat_*_frame), 10 Hz each
  with standalone-receiver noise. Replaces the single navsat.
- web_teleop: turns the Teleop panel's directional pad into car commands,
  like a cruise control. The pad sends one direction at a time, which
  cannot steer a moving car. Hold up/down to raise/lower the target speed
  (it stays); holding down stops at 0 and a new press reverses. Hold
  left/right to turn at the current speed (0.15 1/m). Publishes cmd_vel
  only while in use or moving, so other controllers can drive otherwise.
  Checked with the browser panel: 20 Hz pad messages, speed rises 2 m/s/s.

Co-Authored-By: Claude Opus 5.5 <noreply@anthropic.com>

File: urdf/roof_rack.urdf.xacro (robot description, xacro)
@@ -3,5 +3,5 @@
   Aluminium-profile roof rack that carries the sensors: a rectangular frame on feet with a
   cross bar through the middle, a post on the cross bar for the lidar, a ball head for the
-  camera and two GNSS antenna pucks at the ends of the front bar. Visual only (no
+  camera and two GNSS antenna pucks at opposite corners. Visual only (no
   collisions), with a small mass.
   The rack frame "roof_rack" sits in the middle of the rack, on the top of the profiles
@@ -10,5 +10,5 @@
 -->
 <robot xmlns:xacro="http://ros.org/wiki/xacro">
-    <xacro:macro name="roof_rack" params="parent_link roof_z front_x rear_x half_width clearance profile post_height antenna_y">
+    <xacro:macro name="roof_rack" params="parent_link roof_z front_x rear_x half_width clearance profile post_height antenna1_xy antenna2_xy">
         <xacro:property name="length" value="${front_x - rear_x}" />
         <!-- Rack frame in the parent's coordinates -->
@@ -56,21 +56,17 @@
                 <material name="rack_black" />
             </visual>
-            <!-- GNSS antenna pucks on blocks at both ends of the front bar -->
-            <xacro:rack_box xyz="${front} ${antenna_y} 0.02" size="0.06 0.06 0.04" material="rack_plastic" />
-            <xacro:rack_box xyz="${front} ${-antenna_y} 0.02" size="0.06 0.06 0.04" material="rack_plastic" />
-            <visual>
-                <origin xyz="${front} ${antenna_y} 0.055" rpy="0 0 0" />
-                <geometry>
-                    <cylinder radius="0.04" length="0.03" />
-                </geometry>
-                <material name="rack_black" />
-            </visual>
-            <visual>
-                <origin xyz="${front} ${-antenna_y} 0.055" rpy="0 0 0" />
-                <geometry>
-                    <cylinder radius="0.04" length="0.03" />
-                </geometry>
-                <material name="rack_black" />
-            </visual>
+            <!-- GNSS antenna pucks on blocks (antenna*_xy: x y in the rack frame) -->
+            <xacro:macro name="antenna_puck" params="xy">
+                <xacro:rack_box xyz="${xy} 0.02" size="0.06 0.06 0.04" material="rack_plastic" />
+                <visual>
+                    <origin xyz="${xy} 0.055" rpy="0 0 0" />
+                    <geometry>
+                        <cylinder radius="0.04" length="0.03" />
+                    </geometry>
+                    <material name="rack_black" />
+                </visual>
+            </xacro:macro>
+            <xacro:antenna_puck xy="${antenna1_xy}" />
+            <xacro:antenna_puck xy="${antenna2_xy}" />
             <xacro:inertial_cuboid_with_pose mass="8.0" x="${length}" y="${2 * half_width}" z="${profile}">
                 <origin xyz="0 0 ${bar_z}" rpy="0 0 0" />

File: urdf/sac.urdf.xacro (robot description, xacro)
@@ -63,7 +63,10 @@
   <xacro:property name="lidar_base_above_roof" value="0.20" />
   <xacro:property name="lidar_xyz" value="0 0 ${roof_z + lidar_base_above_roof - rack_top_z + 0.0377}" />
-  <!-- GNSS antennas at both ends of the front bar; the simulated receiver uses the left one -->
+  <!-- Two GNSS antennas at opposite corners of the rack: front right and rear left -->
+  <xacro:property name="rack_rear" value="${rack_rear_x - rack_mid_x}" />    <!-- rear bar, in the rack frame -->
   <xacro:property name="gnss_antenna_y" value="${rack_half_width - 0.03}" />
-  <xacro:property name="gnss_xyz" value="${rack_front} ${gnss_antenna_y} 0.07" />
+  <xacro:property name="gnss_front_right_xy" value="${rack_front} ${-gnss_antenna_y}" />
+  <xacro:property name="gnss_rear_left_xy" value="${rack_rear} ${gnss_antenna_y}" />
+  <xacro:property name="gnss_antenna_z" value="0.07" />   <!-- antenna phase centre above the rack -->
   <!-- Three IMUs on the chassis, on the centre line (not measured): in the middle of the
        car, over the front axle and over the rear axle -->
@@ -177,5 +180,5 @@
     rear_x="${rack_rear_x}" half_width="${rack_half_width}" clearance="${rack_clearance}"
     profile="${rack_profile}" post_height="${roof_z + lidar_base_above_roof - rack_top_z}"
-    antenna_y="${gnss_antenna_y}" />
+    antenna1_xy="${gnss_front_right_xy}" antenna2_xy="${gnss_rear_left_xy}" />
   <xacro:zed2 name="front_camera" parent_link="roof_rack" namespace="$(arg namespace)">
     <origin xyz="${camera_xyz}" rpy="0 ${camera_pitch} 0" />
@@ -190,7 +193,10 @@
     <origin xyz="${back_imu_xyz}" rpy="0 0 0" />
   </xacro:imu>
-  <!-- 10 Hz like a typical GNSS receiver -->
-  <xacro:navsat name="navsat" parent_link="roof_rack" namespace="$(arg namespace)" update_rate="10">
-    <origin xyz="${gnss_xyz}" rpy="0 0 0" />
+  <!-- One fix per antenna at 10 Hz; the heading follows from the two positions -->
+  <xacro:navsat name="navsat_front_right" parent_link="roof_rack" namespace="$(arg namespace)" update_rate="10">
+    <origin xyz="${gnss_front_right_xy} ${gnss_antenna_z}" rpy="0 0 0" />
+  </xacro:navsat>
+  <xacro:navsat name="navsat_rear_left" parent_link="roof_rack" namespace="$(arg namespace)" update_rate="10">
+    <origin xyz="${gnss_rear_left_xy} ${gnss_antenna_z}" rpy="0 0 0" />
   </xacro:navsat>
   <xacro:lidar3d name="roof_lidar" parent_link="roof_rack" namespace="$(arg namespace)">
