Commit message: fix: fast steering response; lower GNSS noise for now
The Ackermann plugin's steering P gain defaulted to 1 (a 1 s time constant), which
made path following weave at 10 m/s; 8 gives ~0.13 s, like power steering.
GNSS noise 0.3 m / 0.5 m until the localization (EKF) is in; the real receiver is
about 1 m / 1.5 m.

Co-Authored-By: Claude Opus 5.5 <noreply@anthropic.com>

File: urdf/sac.gazebo.xacro (robot description, xacro)
@@ -60,4 +60,8 @@
       <kingpin_width>${front_track}</kingpin_width>
       <steering_limit>${steering_limit}</steering_limit>
+      <!-- The steering joints follow the steering angle with this P gain: the default 1 is a
+           1 s time constant, far slower than power steering, and made path following weave
+           at speed. 8 is ~0.13 s. -->
+      <steer_p_gain>8.0</steer_p_gain>
       <wheel_base>${wheel_base}</wheel_base>
       <wheel_separation>${rear_track}</wheel_separation>

File: urdf/sensors.gazebo.xacro (robot description, xacro)
@@ -64,9 +64,11 @@
     </xacro:macro>
     <!-- ============================== GNSS ============================== -->
-    <!-- Error of a standalone (non-RTK) GNSS receiver. Gazebo adds the horizontal noise to
-         latitude and longitude in degrees, so it is converted from metres here. Needs
-         <spherical_coordinates> in the world for real latitude/longitude. -->
-    <xacro:property name="gnss_horizontal_noise" value="1.0" />   <!-- [m] -->
-    <xacro:property name="gnss_vertical_noise" value="1.5" />     <!-- [m] -->
+    <!-- GNSS error. Gazebo adds the horizontal noise to latitude and longitude in degrees, so
+         it is converted from metres here. Needs <spherical_coordinates> in the world for
+         real latitude/longitude.
+         For now lower than the real car's standalone (non-RTK) receiver, which is about 1.0 m
+         horizontal and 1.5 m vertical: set those back once the localization (EKF) is in. -->
+    <xacro:property name="gnss_horizontal_noise" value="0.3" />   <!-- [m] -->
+    <xacro:property name="gnss_vertical_noise" value="0.5" />     <!-- [m] -->
     <xacro:property name="gnss_velocity_noise" value="0.05" />    <!-- [m/s] -->
     <xacro:property name="metres_per_degree" value="111320.0" />

Commit message: feat: suspension in Gazebo; GNSS back to 1 m; track drawn with a localization
- the car's springs (Gazebo joint springs) on sac_description's suspension joints,
  on by default (suspension:=false for the rigid car). The car no longer takes off
  over Sonoma's crests at 10 m/s.
- GNSS noise back to a standalone receiver's 1 m / 1.5 m (localization is in)
- the track marker is frame_locked: with ground_truth_tf:=false there is no
  map -> odom at its zero stamp and viewers did not draw it

Co-Authored-By: Claude Opus 5.5 <noreply@anthropic.com>

File: urdf/sac.gazebo.xacro (robot description, xacro)
@@ -10,6 +10,25 @@
   <xacro:arg name="namespace" default="sac" />
   <xacro:property name="namespace" value="$(arg namespace)" />
+  <!-- Springs and dampers on the wheels (sac_description's suspension); false: a rigid car -->
+  <xacro:arg name="suspension" default="true" />
   <xacro:include filename="$(find sac_description)/urdf/sac.urdf.xacro" />
   <xacro:include filename="$(find gazebo_environment)/urdf/sensors.gazebo.xacro" />
+  <!-- ============================== Suspension ============================== -->
+  <!-- The damper is the joint's damping (sac_description); the spring is Gazebo's joint
+       spring. Its natural length makes the corner load compress it to the middle of the
+       travel at rest, so the ride height is the description's. -->
+  <xacro:macro name="suspension_spring" params="corner sprung_mass">
+    <xacro:property name="stiffness" value="${sprung_mass * (2 * pi * suspension_frequency) ** 2}" />
+    <gazebo reference="${corner}_suspension_joint">
+      <springStiffness>${stiffness}</springStiffness>
+      <springReference>${-sprung_mass * 9.80665 / stiffness}</springReference>
+    </gazebo>
+  </xacro:macro>
+  <xacro:if value="${suspension}">
+    <xacro:suspension_spring corner="front_left" sprung_mass="${front_corner_mass}" />
+    <xacro:suspension_spring corner="front_right" sprung_mass="${front_corner_mass}" />
+    <xacro:suspension_spring corner="rear_left" sprung_mass="${rear_corner_mass}" />
+    <xacro:suspension_spring corner="rear_right" sprung_mass="${rear_corner_mass}" />
+  </xacro:if>
   <!-- ============================== Tyres ============================== -->
   <xacro:macro name="tyre" params="wheel">

File: urdf/sensors.gazebo.xacro (robot description, xacro)
@@ -64,11 +64,9 @@
     </xacro:macro>
     <!-- ============================== GNSS ============================== -->
-    <!-- GNSS error. Gazebo adds the horizontal noise to latitude and longitude in degrees, so
-         it is converted from metres here. Needs <spherical_coordinates> in the world for
-         real latitude/longitude.
-         For now lower than the real car's standalone (non-RTK) receiver, which is about 1.0 m
-         horizontal and 1.5 m vertical: set those back once the localization (EKF) is in. -->
-    <xacro:property name="gnss_horizontal_noise" value="0.3" />   <!-- [m] -->
-    <xacro:property name="gnss_vertical_noise" value="0.5" />     <!-- [m] -->
+    <!-- Error of a standalone (non-RTK) GNSS receiver like the real car's. Gazebo adds the
+         horizontal noise to latitude and longitude in degrees, so it is converted from metres
+         here. Needs <spherical_coordinates> in the world for real latitude/longitude. -->
+    <xacro:property name="gnss_horizontal_noise" value="1.0" />   <!-- [m] -->
+    <xacro:property name="gnss_vertical_noise" value="1.5" />     <!-- [m] -->
     <xacro:property name="gnss_velocity_noise" value="0.05" />    <!-- [m/s] -->
     <xacro:property name="metres_per_degree" value="111320.0" />

Commit message: feat: tyre slip and grip presets
- Gazebo's WheelSlip on the four wheels: slip grows with the force on the tyre
  instead of full grip up to the friction limit (1.2 deg slip angle in Sonoma's
  corners at 10 m/s on dry tyres, 1.7 deg on wet)
- the first friction direction (fdir1) is the axle: mu1 lateral, mu2 longitudinal
- tyre:=dry|wet|gravel presets; each value (tyre_mu_longitudinal, tyre_mu_lateral,
  tyre_slip_longitudinal, tyre_slip_lateral) can be set on its own; sonoma.launch.py
  passes tyre:= and xacro_args:= to the car's xacro

Laps at 10 m/s driven on sac_localization: dry 0.21 m, wet 0.25 m mean error.

Co-Authored-By: Claude Opus 5.5 <noreply@anthropic.com>

File: urdf/sac.gazebo.xacro (robot description, xacro)
@@ -32,8 +32,43 @@
   </xacro:if>
   <!-- ============================== Tyres ============================== -->
+  <!-- Grip and slip of the tyres on the ground.
+         tyre:=dry|wet|gravel                a preset (default dry)
+         tyre_mu_longitudinal:=, tyre_mu_lateral:=
+                                             friction coefficients, driving/braking and sideways
+         tyre_slip_longitudinal:=, tyre_slip_lateral:=
+                                             slip compliance (Gazebo's WheelSlip): how much the
+                                             tyre slips per unit of force/load; the slip angle
+                                             [rad] is about lateral compliance x (lateral force /
+                                             load), so 0.1 is ~3 deg at half the grip, a road tyre
+       Each value overrides the preset's; from the launch file: xacro_args:="tyre_mu_lateral:=0.8". -->
+  <xacro:arg name="tyre" default="dry" />
+  <xacro:arg name="tyre_mu_longitudinal" default="" />
+  <xacro:arg name="tyre_mu_lateral" default="" />
+  <xacro:arg name="tyre_slip_longitudinal" default="" />
+  <xacro:arg name="tyre_slip_lateral" default="" />
+  <xacro:property name="tyre" value="$(arg tyre)" />
+  <!-- Presets: [mu longitudinal, mu lateral, slip longitudinal, slip lateral]. An unknown name
+       fails with "tyre_preset not defined". -->
+  <xacro:if value="${tyre == 'dry'}">
+    <xacro:property name="tyre_preset" value="${[1.1, 1.0, 0.05, 0.1]}" />
+  </xacro:if>
+  <xacro:if value="${tyre == 'wet'}">
+    <xacro:property name="tyre_preset" value="${[0.7, 0.6, 0.08, 0.15]}" />
+  </xacro:if>
+  <xacro:if value="${tyre == 'gravel'}">
+    <xacro:property name="tyre_preset" value="${[0.55, 0.5, 0.15, 0.3]}" />
+  </xacro:if>
+  <xacro:property name="tyre_mu_longitudinal" value="${float('$(arg tyre_mu_longitudinal)' or tyre_preset[0])}" />
+  <xacro:property name="tyre_mu_lateral" value="${float('$(arg tyre_mu_lateral)' or tyre_preset[1])}" />
+  <xacro:property name="tyre_slip_longitudinal" value="${float('$(arg tyre_slip_longitudinal)' or tyre_preset[2])}" />
+  <xacro:property name="tyre_slip_lateral" value="${float('$(arg tyre_slip_lateral)' or tyre_preset[3])}" />
+  <!-- fdir1 is the first friction direction in the wheel link's frame: its z axis, the axle.
+       So mu1 is the sideways grip and mu2 the grip along the tyre, whichever way the wheel
+       turns or steers (and WheelSlip's lateral slip goes with fdir1 too). -->
   <xacro:macro name="tyre" params="wheel">
     <gazebo reference="${wheel}">
-      <mu1>1.1</mu1>
-      <mu2>1.1</mu2>
+      <mu1>${tyre_mu_lateral}</mu1>
+      <mu2>${tyre_mu_longitudinal}</mu2>
+      <fdir1>0 0 1</fdir1>
     </gazebo>
   </xacro:macro>
@@ -42,4 +77,24 @@
   <xacro:tyre wheel="rear_left_wheel" />
   <xacro:tyre wheel="rear_right_wheel" />
+  <!-- Slip grows with the force on the tyre, like a real one, instead of full grip up to the
+       friction limit. The load is the corner's weight at rest. -->
+  <xacro:macro name="wheel_slip" params="wheel load">
+    <wheel link_name="${wheel}">
+      <slip_compliance_longitudinal>${tyre_slip_longitudinal}</slip_compliance_longitudinal>
+      <slip_compliance_lateral>${tyre_slip_lateral}</slip_compliance_lateral>
+      <wheel_normal_force>${load}</wheel_normal_force>
+      <wheel_radius>${wheel_radius}</wheel_radius>
+    </wheel>
+  </xacro:macro>
+  <xacro:property name="front_wheel_load" value="${(front_corner_mass + suspension_mass + wheel_mass + 1.0) * 9.80665}" />
+  <xacro:property name="rear_wheel_load" value="${(rear_corner_mass + suspension_mass + wheel_mass) * 9.80665}" />
+  <gazebo>
+    <plugin filename="gz-sim-wheel-slip-system" name="gz::sim::systems::WheelSlip">
+      <xacro:wheel_slip wheel="front_left_wheel" load="${front_wheel_load}" />
+      <xacro:wheel_slip wheel="front_right_wheel" load="${front_wheel_load}" />
+      <xacro:wheel_slip wheel="rear_left_wheel" load="${rear_wheel_load}" />
+      <xacro:wheel_slip wheel="rear_right_wheel" load="${rear_wheel_load}" />
+    </plugin>
+  </gazebo>
   <!-- ============================== Sensors ============================== -->
   <!-- Keep the rack as its own link, so the sensors hang off it -->

Commit message: feat: see-through ground truth car in the viewer; springs and tyres on the whole car's load
- ground_truth_marker: a translucent copy of the car at Gazebo's exact pose
  (/sac/ground_truth/marker, in the map frame), to compare with a localization
- wheel loads for WheelSlip and the spring preload from sac_description's car_mass

Co-Authored-By: Claude Opus 5.5 <noreply@anthropic.com>

File: urdf/sac.gazebo.xacro (robot description, xacro)
@@ -16,6 +16,7 @@
   <!-- ============================== Suspension ============================== -->
   <!-- The damper is the joint's damping (sac_description); the spring is Gazebo's joint
-       spring. Its natural length makes the corner load compress it to the middle of the
-       travel at rest, so the ride height is the description's. -->
+       spring. Its natural length makes the corner load (the whole car's weight on that
+       corner) compress it to the middle of the travel at rest, so the car and its sensors
+       stand at the description's height. -->
   <xacro:macro name="suspension_spring" params="corner sprung_mass">
     <xacro:property name="stiffness" value="${sprung_mass * (2 * pi * suspension_frequency) ** 2}" />
@@ -87,6 +88,6 @@
     </wheel>
   </xacro:macro>
-  <xacro:property name="front_wheel_load" value="${(front_corner_mass + suspension_mass + wheel_mass + 1.0) * 9.80665}" />
-  <xacro:property name="rear_wheel_load" value="${(rear_corner_mass + suspension_mass + wheel_mass) * 9.80665}" />
+  <xacro:property name="front_wheel_load" value="${front_corner_mass * 9.80665}" />
+  <xacro:property name="rear_wheel_load" value="${rear_corner_mass * 9.80665}" />
   <gazebo>
     <plugin filename="gz-sim-wheel-slip-system" name="gz::sim::systems::WheelSlip">

Commit message: feat: front 2D lidar and static obstacles along the route
Co-Authored-By: Claude Opus 5.5 <noreply@anthropic.com>

File: urdf/sac.gazebo.xacro (robot description, xacro)
@@ -109,4 +109,5 @@
   <xacro:navsat_gazebo name="navsat_rear_left" namespace="${namespace}" />
   <xacro:vlp16_gazebo name="roof_lidar" namespace="${namespace}" />
+  <xacro:lidar_2d_gazebo name="front_lidar" namespace="${namespace}" />
   <!-- ============================== Gazebo systems ============================== -->
   <!-- Ground truth pose of the whole model, used by the odometry_tf node -->

File: urdf/sensors.gazebo.xacro (robot description, xacro)
@@ -140,4 +140,43 @@
                         <mean>0.0</mean>
                         <stddev>${lidar_noise}</stddev>
+                    </noise>
+                </lidar>
+            </sensor>
+        </gazebo>
+        <xacro:preserve_joint joint="${name}_joint" />
+    </xacro:macro>
+    <!-- ============================== 2D lidar ============================== -->
+    <!-- A generic planar scanner: 180 deg ahead at 0.25 deg, 20 Hz, 30 m, +-2 cm (the front
+         half only: behind it is the car). Publishes <namespace>/sensors/<name>/scan -->
+    <xacro:macro name="lidar_2d_gazebo" params="name namespace update_rate:=20 samples:=721
+        min_angle:=${-pi / 2} max_angle:=${pi / 2} min_range:=0.1 max_range:=30.0 noise:=0.02">
+        <gazebo reference="${name}_frame">
+            <sensor name="${name}_sensor" type="gpu_lidar">
+                <always_on>true</always_on>
+                <update_rate>${update_rate}</update_rate>
+                <gz_frame_id>${name}_frame</gz_frame_id>
+                <topic>${namespace}/sensors/${name}/scan</topic>
+                <lidar>
+                    <scan>
+                        <horizontal>
+                            <samples>${samples}</samples>
+                            <min_angle>${min_angle}</min_angle>
+                            <max_angle>${max_angle}</max_angle>
+                        </horizontal>
+                        <vertical>
+                            <samples>1</samples>
+                            <min_angle>0</min_angle>
+                            <max_angle>0</max_angle>
+                        </vertical>
+                    </scan>
+                    <range>
+                        <min>${min_range}</min>
+                        <max>${max_range}</max>
+                        <resolution>0.01</resolution>
+                    </range>
+                    <noise>
+                        <type>gaussian</type>
+                        <mean>0.0</mean>
+                        <stddev>${noise}</stddev>
                     </noise>
                 </lidar>
